File: EAGLE/Projects/Coilgun/Inverter/Inverter.sch (EAGLE design)
At the start: 18 parts, among them IC1 LM555CN, J1 XT30PW-M, J2 XT30PW-F, Q1 IRF840, Q2 IRF9530, Q3 IRF840, Q4 IRF9530, U1 MIC4422, U2 MIC4421

Commit message: Rename accordingly
Parts:
- added JP1: (no value), pinhead:PINHD-1X2
Connections:
- net N$8 renamed CLOCK
Other:
- moved on the sheet: C1, C2, C33, IC1, R1, R2

Commit message: Add latest mods
Parts:
- removed JP1: (no value), pinhead:PINHD-1X2
- added CLK_555, CLK_EXT: (no value), pinhead:PINHD-1X2
- added D1: 1N4148DO35-7, diode:1N4148DO35-7
- added D2: (no value), diode:ZENER-DIODEDO35Z10
- added F1: 0.2 A, rcl:R-EU_M1206
- added J3: XT30PW-M, XT30PW-M:XT30PW-M
- added X1: SMA-142-0711-871/876, con-coax:SMA-142-0711-871/876
Connections:
- net N$10 renamed DRIVE_INV
- net N$9 renamed DRIVE_NON
- removed net CLOCK: IC1.OUTPUT, U1.IN, U2.IN
- new net CLK: CLK_555.2, CLK_EXT.2, U1.IN, U2.IN
- new net CLK_555: CLK_555.1, IC1.OUTPUT
- new net CLK_EXT: CLK_EXT.1, X1.1
- new net N$11: F1.1, J1.+
- new net VS: J3.+, Q2.S, Q4.S
- net GND: now also D1.A, D2.A, J3.-, X1.2
- net VCC: now also D1.C, D2.C, F1.2; no longer J1.+, Q2.S, Q4.S
Other:
- note added: "Clock generation"
- note added: "Clock selection"
- note added: "Mosfet"
- note added: "Mosfet driver"
- note added: "OV protection"
- note added: "Protection"
- note added: "Reverse protection"
- moved on the sheet: C1, C2, C3, C33, C4, C5, C6, IC1, J1, J2, Q1, Q2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
